File: KiCAD/nanopad.sch (KiCad schematic (older format))
At the start: 130 parts, among them J1 CONN_01X03_MALE, J2 CONN_01X03_MALE, J3 CONN_02X10, P1 SERVO, P2 SERVO, Q1 Crystal_3.2x1.5, Q2 Crystal_3.2x1.5, Q3 3904, Q4 3904, Q5 3904, Q6 3904, SW1 SW_Push, SW10 Left, SW2 SW_Push, SW3 Up, SW4 Up, SW5 Right, SW6 Right, SW7 Down, SW8 Down, SW9 Left, U1 LM1117-3.3, U2 LM1117-3.3, U3 MMA8653FCR1, U4 MMA8653FCR1, U5 STM32F401RETx, U6 STM32F401RETx, U7 MCP9700AT-E/LT, U8 MCP9700AT-E/LT, U9 MC74VHC1GT125, Y1 Crystal_3.2x2.5, Y2 Crystal_3.2x2.5, Y3 Crystal_12Mhz, Y4 Crystal_12Mhz

Commit message: fixing electrical rules error
ok
Parts:
- removed C10, C13, C3, C4: .1uf, symbol CP1
- removed C15: CP1, symbol CP1
- removed C17, C23: 27pf, symbol CP1
- removed C19, C25, C32: .1uF, symbol CP1
- removed C21, C6: 22uF, symbol CP1
- removed C28, C30: 4.7uF, symbol CP1
- removed C34: 2.2uF, symbol CP1
- removed D1: RED_PWR, symbol LED_Small
- removed D10, D6, D8: LED, symbol LED
- removed D12: ZHCS400, symbol DIODESCH
- removed D4: LED_RGB, symbol LED_RGB
- removed J2: CONN_01X03_MALE, symbol CONN_01X03_MALE
- removed P2: SERVO, symbol SERVO
- removed Q4: 3904, TO_SOT_Packages_THT:TO-220_Vertical, symbol 2SC1945
- removed R12, R14: 2.2K, symbol R
- removed R16, R32, R34, R36, R38, R9: 10K, symbol R
- removed R18, R20, R22, R24, R26, R28, R4: 330, symbol R
- removed R30: R_PHOTO, symbol R_PHOTO
- removed R41: 470, symbol R
- removed R6: 15K, symbol R
- removed SW10: Left, symbol SW_Push
- removed SW2: SW_Push, symbol SW_Push
- removed SW4: Up, symbol SW_Push
- removed SW6: Right, symbol SW_Push
- removed SW8: Down, symbol SW_Push
- removed U1: LM1117-3.3, symbol LM1117-3.3
- removed U4: MMA8653FCR1, DFN10, symbol MMA8653FCR1
- removed U5: STM32F401RETx, LQFP64, symbol STM32F401RETx
- removed U8: MCP9700AT-E/LT, TO_SOT_Packages_SMD:SC-70-5, symbol MCP9700AT-E/LT
- removed Y1: Crystal_3.2x2.5, symbol Crystal
- removed Y3: Crystal_12Mhz, symbol Crystal
- added F1: 1206L025YR, symbol Fuse
- renumbered C11 to C10, C2 to C11, C5 to C2, C7 to C4, C8 to C6, C1 to C7, C9 to C8, Q2 to Q1, Q1 to Q2, R3 to R1, R5 to R3, R1 to R5, R7 to R6, R2 to R7
Connections:
- net labels removed: RC9_RGB_R
- wire segments 267 -> 270
- no-connect marks 0 -> 8
Other:
- moved on the sheet: D3, R17, R19, R21

Commit message: reset anotation
ok
Parts:
- removed R6, R8: 33, symbol R
- renumbered C2 to C1, C16 to C10, C18 to C11, C20 to C12, C22 to C13, C24 to C14, C26 to C15, C27 to C16, C29 to C17, C31 to C18, C33 to C19, C4 to C2, C35 to C20, C6 to C3, C7 to C4, C8 to C5, C10 to C6, C11 to C7, C12 to C8, C14 to C9, D2 to D1, D3 to D2, D5 to D3, D7 to D4, D9 to D5, D11 to D6, J3 to J2, Q5 to Q4, Q6 to Q5, R19 to R10, R21 to R11, R23 to R12, R25 to R13, R27 to R14, R29 to R15, R31 to R16, R33 to R17, R35 to R18, R37 to R19, R3 to R2, R39 to R20, R40 to R21, R42 to R22, R43 to R23, R44 to R24, R45 to R25, R5 to R3, R7 to R4, R10 to R5, R11 to R6, R13 to R7, R15 to R8, R17 to R9, SW3 to SW2, SW5 to SW3, SW7 to SW4, SW9 to SW5, U2 to U1, U3 to U2, U6 to U3, U7 to U4, U9 to U5, Y2 to Y1, Y4 to Y2
